File: alarm_circuit/alarm_circuit.kicad_sch (KiCad schematic)
At the start: 13 parts, among them J1 Screw_Terminal_01x03, J2 Screw_Terminal_01x03, J3 DIN-5_180degree, J4 Screw_Terminal_01x04, K1 FINDER-40.52, Q1 BC547, SW1 SW_Push, U1 NodeMCU-ESP8266

Commit message: added deactivation button to circuit
Parts:
- added R3: 1M, symbol Device:R
- added SW2: SW_Push, symbol Switch:SW_Push
Connections:
- net DIN5-Pin3: now also SW2.1
- net GND: now also R3.1
- net at U1.23 (D5): now also R3.2, SW2.2
- no-connect marks 19 -> 18
